File: DaughterBoard_STM32F4DISCO.kicad_pcb (KiCad board)
At the start: 2 copper layers, 33 parts, among them P1 TYP2A_SPI1, P10 TYP2_SPI3, P11 TYP2_SPI4, P12 I2C1, P13 I2C2, P14 I2C3, P15 TYP3_UART1, P16 TYP3_UART2, P17 TYP3_UART6, P18 TYP1_GPIO1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

Commit message: Added a few resources
Parts:
- P1, P2, P21, P3, P4: footprint Pin_Headers.pretty:Pin_Header_Straight_2x06 -> Socket_Strips.pretty:Socket_Strip_Straight_2x06
- P10, P11, P15, P16, P17, P18, P19, P20, P22, P23, P8, P9: footprint Pin_Headers.pretty:Pin_Header_Straight_1x06 -> Socket_Strips.pretty:Socket_Strip_Straight_1x06
- P12, P13, P14, P5, P6, P7: footprint Pin_Headers.pretty:Pin_Header_Straight_1x04 -> Socket_Strips.pretty:Socket_Strip_Straight_1x04
- P24, P26: footprint Pin_Headers.pretty:Pin_Header_Straight_1x02 -> Socket_Strips.pretty:Socket_Strip_Straight_1x02
- P25, P27: footprint Pin_Headers.pretty:Pin_Header_Straight_2x25 -> Socket_Strips.pretty:Socket_Strip_Straight_2x25
- moved P16 124.6 mm to (47.0, 84.0), turned to 90 degrees
- moved P8 118.8 mm to (40.0, 104.0), turned to 90 degrees
- moved P1 113.5 mm to (34.0, 158.0), turned to 90 degrees
- moved P12 112.5 mm to (32.0, 141.0), turned to 90 degrees
- moved P18 112.4 mm to (36.0, 124.0), turned to 90 degrees
- moved P21 111.7 mm to (64.0, 84.0), turned to 90 degrees
- moved P15 105.2 mm to (39.0, 84.0), turned to 90 degrees
- moved P5 104.8 mm to (40.0, 141.0), turned to 90 degrees
- moved P9 96.8 mm to (48.0, 104.0), turned to 90 degrees
- moved P6 96.0 mm to (48.0, 141.0), turned to 90 degrees
- moved P19 95.4 mm to (44.0, 124.0), turned to 90 degrees
- moved P3 93.2 mm to (58.0, 158.0), turned to 90 degrees
- moved P17 88.9 mm to (55.0, 84.0), turned to 90 degrees
- moved P13 88.3 mm to (56.0, 141.0), turned to 90 degrees
- moved P10 86.8 mm to (56.0, 104.0), turned to 90 degrees
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Routing:
- net /PD4: track 0.00 -> 33.4 mm, vias 0 -> 1
- net /PD3: track 0.00 -> 32.0 mm, vias 0 -> 1
- net /PD7: track 0.00 -> 26.1 mm
- net /PE2: track 0.00 -> 24.8 mm, vias 0 -> 1
- net /PE5: track 0.00 -> 21.7 mm
- net /PE6: track 0.00 -> 16.0 mm
- net (no net): track 0.00 -> 15.5 mm
