File: DaughterBoard_STM32F4DISCO.sch (KiCad schematic (older format))
At the start: 33 parts, among them P1 CONN_02X06, P10 CONN_01X06, P11 CONN_01X06, P12 CONN_01X04, P13 CONN_01X04, P14 CONN_01X04, P15 CONN_01X06, P16 CONN_01X06, P17 CONN_01X06, P18 CONN_01X06, P19 CONN_01X06, P2 CONN_02X06, P20 CONN_01X06, P21 CONN_02X06, P22 CONN_01X06, P23 CONN_01X06, P24 CONN_01X02, P25 CONN_02X25, P26 CONN_01X02, P27 CONN_02X25, P3 CONN_02X06, P4 CONN_02X06, P5 CONN_01X04, P6 CONN_01X04, P7 CONN_01X04, P8 CONN_01X06, P9 CONN_01X06

Commit message: Schematic complete Layout placement half done.
Parts:
- D1, D2, D3: footprint (none) -> LEDs.pretty:LED-0603
- P1: value CONN_02X06 -> TYP2A_SPI1; footprint (none) -> Pin_Headers.pretty:Pin_Header_Straight_2x06
- P10: value CONN_01X06 -> TYP2_SPI3; footprint (none) -> Pin_Headers.pretty:Pin_Header_Straight_1x06
- P11: value CONN_01X06 -> TYP2_SPI4; footprint (none) -> Pin_Headers.pretty:Pin_Header_Straight_1x06
- P12, P5: value CONN_01X04 -> I2C1; footprint (none) -> Pin_Headers.pretty:Pin_Header_Straight_1x04
- P13, P6: value CONN_01X04 -> I2C2; footprint (none) -> Pin_Headers.pretty:Pin_Header_Straight_1x04
- P14, P7: value CONN_01X04 -> I2C3; footprint (none) -> Pin_Headers.pretty:Pin_Header_Straight_1x04
- P15: value CONN_01X06 -> TYP3_UART1; footprint (none) -> Pin_Headers.pretty:Pin_Header_Straight_1x06
- P16: value CONN_01X06 -> TYP3_UART2; footprint (none) -> Pin_Headers.pretty:Pin_Header_Straight_1x06
- P17: value CONN_01X06 -> TYP3_UART6; footprint (none) -> Pin_Headers.pretty:Pin_Header_Straight_1x06
- P18: value CONN_01X06 -> TYP1_GPIO1; footprint (none) -> Pin_Headers.pretty:Pin_Header_Straight_1x06
- P19: value CONN_01X06 -> TYP1_GPIO2; footprint (none) -> Pin_Headers.pretty:Pin_Header_Straight_1x06
- P2: value CONN_02X06 -> TYP2A_SPI2; footprint (none) -> Pin_Headers.pretty:Pin_Header_Straight_2x06
- P20: value CONN_01X06 -> TYP1_GPIO3; footprint (none) -> Pin_Headers.pretty:Pin_Header_Straight_1x06
- P21: value CONN_02X06 -> TIM1; footprint (none) -> Pin_Headers.pretty:Pin_Header_Straight_2x06
- P22: value CONN_01X06 -> TYP1_GPIO4; footprint (none) -> Pin_Headers.pretty:Pin_Header_Straight_1x06
- P23: value CONN_01X06 -> TYP1_GPIO5; footprint (none) -> Pin_Headers.pretty:Pin_Header_Straight_1x06
- P24, P26: footprint (none) -> Pin_Headers.pretty:Pin_Header_Straight_1x02
- P25, P27: footprint (none) -> Pin_Headers.pretty:Pin_Header_Straight_2x25
- P3: value CONN_02X06 -> TYP2A_SPI3; footprint (none) -> Pin_Headers.pretty:Pin_Header_Straight_2x06
- P4: value CONN_02X06 -> TYP2A_SPI4; footprint (none) -> Pin_Headers.pretty:Pin_Header_Straight_2x06
- P8: value CONN_01X06 -> TYP2_SPI1; footprint (none) -> Pin_Headers.pretty:Pin_Header_Straight_1x06
- P9: value CONN_01X06 -> TYP2_SPI2; footprint (none) -> Pin_Headers.pretty:Pin_Header_Straight_1x06
- R1, R2, R3: footprint (none) -> Resistors_SMD.pretty:R_0603
Connections:
- net BOOT0: now also P27.21 (P21); no longer P27.22 (P22)
- net GND: now also P25.23 (P23), P25.5 (P5); no longer P25.24 (P24), P25.6 (P6)
- net NC1: now also P25.48 (P48); no longer P25.47 (P47)
- net NC2: now also P25.35 (P35); no longer P25.36 (P36)
- net NRST: now also P25.6 (P6); no longer P25.5 (P5)
- net PA0: now also P25.12 (P12); no longer P25.11 (P11)
- net PA1: now also P25.11 (P11); no longer P25.12 (P12)
- net PA10: now also P27.41 (P41); no longer P27.42 (P42)
- net PA13: now also P27.42 (P42); no longer P27.41 (P41)
- net PA14: now also P27.39 (P39); no longer P27.40 (P40)
- net PA15: now also P27.40 (P40); no longer P27.39 (P39)
- net PA2: now also P25.14 (P14); no longer P25.13 (P13)
- net PA3: now also P25.13 (P13); no longer P25.14 (P14)
- net PA4: now also P25.16 (P16); no longer P25.15 (P15)
- net PA5: now also P25.15 (P15); no longer P25.16 (P16)
- net PA6: now also P25.18 (P18); no longer P25.17 (P17)
- net PA7: now also P25.17 (P17); no longer P25.18 (P18)
- net PA8: now also P27.43 (P43); no longer P27.44 (P44)
- net PA9: now also P27.44 (P44); no longer P27.43 (P43)
- net PB0: now also P25.22 (P22); no longer P25.21 (P21)
- net PB1: now also P25.21 (P21); no longer P25.22 (P22)
- net PB10: now also P25.34 (P34); no longer P25.33 (P33)
- net PB12: now also P25.36 (P36); no longer P25.35 (P35)
- net PB13: now also P25.37 (P37); no longer P25.38 (P38)
- net PB14: now also P25.38 (P38); no longer P25.37 (P37)
- net PB2: now also P25.24 (P24); no longer P25.23 (P23)
- net PB3: now also P27.28 (P28); no longer P27.27 (P27)
- net PB4: now also P27.25 (P25); no longer P27.26 (P26)
- net PB5: now also P27.26 (P26); no longer P27.25 (P25)
- net PB6: now also P27.23 (P23); no longer P27.24 (P24)
- net PB7: now also P27.24 (P24); no longer P27.23 (P23)
- net PB8: now also P27.19 (P19); no longer P27.20 (P20)
- net PB9: now also P27.20 (P20); no longer P27.19 (P19)
- net PC0: now also P25.8 (P8); no longer P25.7 (P7)
- net PC1: now also P25.7 (P7); no longer P25.8 (P8)
- net PC10: now also P27.37 (P37); no longer P27.38 (P38)
- net PC11: now also P27.38 (P38); no longer P27.37 (P37)
- net PC12: now also P27.35 (P35); no longer P27.36 (P36)
- net PC13: now also P27.12 (P12); no longer P27.11 (P11)
- net PC14: now also P27.9 (P9); no longer P27.10 (P10)
- net PC15: now also P27.10 (P10); no longer P27.9 (P9)
- net PC2: now also P25.10 (P10); no longer P25.9 (P9)
- net PC3: now also P25.9 (P9); no longer P25.10 (P10)
- net PC4: now also P25.20 (P20); no longer P25.19 (P19)
- net PC5: now also P25.19 (P19); no longer P25.20 (P20)
- net PC6: now also P27.47 (P47); no longer P27.48 (P48)
- net PC7: now also P27.48 (P48); no longer P27.47 (P47)
- net PC8: now also P27.45 (P45); no longer P27.46 (P46)
- net PC9: now also P27.46 (P46); no longer P27.45 (P45)
- net PD0: now also P27.36 (P36); no longer P27.35 (P35)
- net PD1: now also P27.33 (P33); no longer P27.34 (P34)
- net PD10: now also P25.42 (P42); no longer P25.41 (P41)
- net PD11: now also P25.43 (P43); no longer P25.44 (P44)
- net PD12: now also P25.44 (P44); no longer P25.43 (P43)
- net PD13: now also P25.45 (P45); no longer P25.46 (P46)
- net PD14: now also P25.46 (P46); no longer P25.45 (P45)
- net PD15: now also P25.47 (P47); no longer P25.48 (P48)
- net PD2: now also P27.34 (P34); no longer P27.33 (P33)
- net PD3: now also P27.31 (P31); no longer P27.32 (P32)
- net PD4: now also P27.32 (P32); no longer P27.31 (P31)
- net PD5: now also P27.29 (P29); no longer P27.30 (P30)
- net PD6: now also P27.30 (P30); no longer P27.29 (P29)
- net PD7: now also P27.27 (P27); no longer P27.28 (P28)
- net PD8: now also P25.40 (P40); no longer P25.39 (P39)
- net PD9: now also P25.41 (P41); no longer P25.42 (P42)
- net PE0: now also P27.17 (P17); no longer P27.18 (P18)
- net PE1: now also P27.18 (P18); no longer P27.17 (P17)
- net PE10: now also P25.28 (P28); no longer P25.27 (P27)
- net PE11: now also P25.29 (P29); no longer P25.30 (P30)
- net PE12: now also P25.30 (P30); no longer P25.29 (P29)
- net PE13: now also P25.31 (P31); no longer P25.32 (P32)
- net PE14: now also P25.32 (P32); no longer P25.31 (P31)
- net PE15: now also P25.33 (P33), P25.39 (P39); no longer P25.34 (P34), P25.40 (P40)
- net PE2: now also P27.15 (P15); no longer P27.16 (P16)
- net PE3: now also P27.16 (P16); no longer P27.15 (P15)
- net PE4: now also P27.13 (P13); no longer P27.14 (P14)
- net PE5: now also P27.14 (P14); no longer P27.13 (P13)
- net PE6: now also P27.11 (P11); no longer P27.12 (P12)
- net PE7: now also P25.25 (P25); no longer P25.26 (P26)
- net PE8: now also P25.26 (P26); no longer P25.25 (P25)
- net PE9: now also P25.27 (P27); no longer P25.28 (P28)
- net PH0: now also P27.7 (P7); no longer P27.8 (P8)
- net PH1: now also P27.8 (P8); no longer P27.7 (P7)
- net VDD: now also P27.22 (P22); no longer P27.21 (P21)
Other:
- note removed: "GPIO1"
- note removed: "GPIO2"
- note removed: "GPIO3"
- note removed: "I2C1"
- note removed: "I2C2"
- note removed: "I2C3"
- note removed: "SPI1"
- note removed: "SPI2"
- note removed: "SPI3"
- note removed: "SPI4"
- note removed: "TIM1\n"
- note removed: "UART1"
- note removed: "UART2"
- note removed: "UART6"

Commit message: Added a few resources
Parts:
- P1, P2, P21, P3, P4: footprint Pin_Headers.pretty:Pin_Header_Straight_2x06 -> Socket_Strips.pretty:Socket_Strip_Straight_2x06
- P10, P11, P15, P16, P17, P18, P19, P20, P22, P23, P8, P9: footprint Pin_Headers.pretty:Pin_Header_Straight_1x06 -> Socket_Strips.pretty:Socket_Strip_Straight_1x06
- P12, P13, P14, P5, P6, P7: footprint Pin_Headers.pretty:Pin_Header_Straight_1x04 -> Socket_Strips.pretty:Socket_Strip_Straight_1x04
- P24, P26: footprint Pin_Headers.pretty:Pin_Header_Straight_1x02 -> Socket_Strips.pretty:Socket_Strip_Straight_1x02
- P25, P27: footprint Pin_Headers.pretty:Pin_Header_Straight_2x25 -> Socket_Strips.pretty:Socket_Strip_Straight_2x25
Changed lines of the file:
@@
 F 0 "P25" H 8550 4000 50  0000 C CNN
 F 1 "CONN_02X25" V 8550 2700 50  0000 C CNN
-F 2 "Pin_Headers.pretty:Pin_Header_Straight_2x25" H 8550 1950 60  0001 C CNN
+F 2 "Socket_Strips.pretty:Socket_Strip_Straight_2x25" H 8550 1950 60  0001 C CNN
 F 3 "" H 8550 1950 60  0000 C CNN
 	1    8550 2700
@@
 F 0 "P27" H 10000 4000 50  0000 C CNN
 F 1 "CONN_02X25" V 10000 2700 50  0000 C CNN
-F 2 "Pin_Headers.pretty:Pin_Header_Straight_2x25" H 10000 1950 60  0001 C CNN
+F 2 "Socket_Strips.pretty:Socket_Strip_Straight_2x25" H 10000 1950 60  0001 C CNN
 F 3 "" H 10000 1950 60  0000 C CNN
 	1    10000 2700
@@
 F 0 "P24" H 8500 1100 50  0000 C CNN
 F 1 "CONN_01X02" V 8600 950 50  0000 C CNN
-F 2 "Pin_Headers.pretty:Pin_Header_Straight_1x02" H 8500 950 60  0001 C CNN
+F 2 "Socket_Strips.pretty:Socket_Strip_Straight_1x02" H 8500 950 60  0001 C CNN
 F 3 "" H 8500 950 60  0000 C CNN
 	1    8500 950
@@
 F 0 "P26" H 9950 1100 50  0000 C CNN
 F 1 "CONN_01X02" V 10050 950 50  0000 C CNN
-F 2 "Pin_Headers.pretty:Pin_Header_Straight_1x02" H 9950 950 60  0001 C CNN
+F 2 "Socket_Strips.pretty:Socket_Strip_Straight_1x02" H 9950 950 60  0001 C CNN
 F 3 "" H 9950 950 60  0000 C CNN
 	1    9950 950
@@
 F 0 "P5" H 1300 6300 50  0000 C CNN
 F 1 "I2C1" V 1400 6050 50  0000 C CNN
-F 2 "Pin_Headers.pretty:Pin_Header_Straight_1x04" H 1300 6050 60  0001 C CNN
+F 2 "Socket_Strips.pretty:Socket_Strip_Straight_1x04" H 1300 6050 60  0001 C CNN
 F 3 "" H 1300 6050 60  0000 C CNN
 	1    1300 6050
@@
 F 0 "P6" H 1300 7000 50  0000 C CNN
 F 1 "I2C2" V 1400 6750 50  0000 C CNN
-F 2 "Pin_Headers.pretty:Pin_Header_Straight_1x04" H 1300 6750 60  0001 C CNN
+F 2 "Socket_Strips.pretty:Socket_Strip_Straight_1x04" H 1300 6750 60  0001 C CNN
 F 3 "" H 1300 6750 60  0000 C CNN
 	1    1300 6750
@@
 F 0 "P7" H 1300 7700 50  0000 C CNN
 F 1 "I2C3" V 1400 7450 50  0000 C CNN
-F 2 "Pin_Headers.pretty:Pin_Header_Straight_1x04" H 1300 7450 60  0001 C CNN
+F 2 "Socket_Strips.pretty:Socket_Strip_Straight_1x04" H 1300 7450 60  0001 C CNN
 F 3 "" H 1300 7450 60  0000 C CNN
 	1    1300 7450
@@
 F 0 "P1" H 1150 2200 50  0000 C CNN
 F 1 "TYP2A_SPI1" H 1150 1500 50  0000 C CNN
-F 2 "Pin_Headers.pretty:Pin_Header_Straight_2x06" H 1150 650 60  0001 C CNN
+F 2 "Socket_Strips.pretty:Socket_Strip_Straight_2x06" H 1150 650 60  0001 C CNN
 F 3 "" H 1150 650 60  0000 C CNN
 	1    1150 1850
@@
 F 0 "P2" H 1150 3100 50  0000 C CNN
 F 1 "TYP2A_SPI2" H 1150 2400 50  0000 C CNN
-F 2 "Pin_Headers.pretty:Pin_Header_Straight_2x06" H 1150 1550 60  0001 C CNN
+F 2 "Socket_Strips.pretty:Socket_Strip_Straight_2x06" H 1150 1550 60  0001 C CNN
 F 3 "" H 1150 1550 60  0000 C CNN
 	1    1150 2750
@@
 F 0 "P3" H 1150 4000 50  0000 C CNN
 F 1 "TYP2A_SPI3" H 1150 3300 50  0000 C CNN
-F 2 "Pin_Headers.pretty:Pin_Header_Straight_2x06" H 1150 2450 60  0001 C CNN
+F 2 "Socket_Strips.pretty:Socket_Strip_Straight_2x06" H 1150 2450 60  0001 C CNN
 F 3 "" H 1150 2450 60  0000 C CNN
 	1    1150 3650
@@
 F 0 "P4" H 1150 4900 50  0000 C CNN
 F 1 "TYP2A_SPI4" H 1150 4200 50  0000 C CNN
-F 2 "Pin_Headers.pretty:Pin_Header_Straight_2x06" H 1150 3350 60  0001 C CNN
+F 2 "Socket_Strips.pretty:Socket_Strip_Straight_2x06" H 1150 3350 60  0001 C CNN
 F 3 "" H 1150 3350 60  0000 C CNN
 	1    1150 4550
@@
 F 0 "P8" H 2600 2200 50  0000 C CNN
 F 1 "TYP2_SPI1" V 2700 1850 50  0000 C CNN
-F 2 "Pin_Headers.pretty:Pin_Header_Straight_1x06" H 2600 1850 60  0001 C CNN
+F 2 "Socket_Strips.pretty:Socket_Strip_Straight_1x06" H 2600 1850 60  0001 C CNN
 F 3 "" H 2600 1850 60  0000 C CNN
 	1    2600 1850
@@
 F 0 "P9" H 2600 3100 50  0000 C CNN
 F 1 "TYP2_SPI2" V 2700 2750 50  0000 C CNN
-F 2 "Pin_Headers.pretty:Pin_Header_Straight_1x06" H 2600 2750 60  0001 C CNN
+F 2 "Socket_Strips.pretty:Socket_Strip_Straight_1x06" H 2600 2750 60  0001 C CNN
 F 3 "" H 2600 2750 60  0000 C CNN
 	1    2600 2750
@@
 F 0 "P10" H 2600 4000 50  0000 C CNN
 F 1 "TYP2_SPI3" V 2700 3650 50  0000 C CNN
-F 2 "Pin_Headers.pretty:Pin_Header_Straight_1x06" H 2600 3650 60  0001 C CNN
+F 2 "Socket_Strips.pretty:Socket_Strip_Straight_1x06" H 2600 3650 60  0001 C CNN
 F 3 "" H 2600 3650 60  0000 C CNN
 	1    2600 3650
@@
 F 0 "P12" H 2600 6300 50  0000 C CNN
 F 1 "I2C1" V 2700 6050 50  0000 C CNN
-F 2 "Pin_Headers.pretty:Pin_Header_Straight_1x04" H 2600 6050 60  0001 C CNN
+F 2 "Socket_Strips.pretty:Socket_Strip_Straight_1x04" H 2600 6050 60  0001 C CNN
 F 3 "" H 2600 6050 60  0000 C CNN
 	1    2600 6050
@@
 F 0 "P13" H 2600 7000 50  0000 C CNN
 F 1 "I2C2" V 2700 6750 50  0000 C CNN
-F 2 "Pin_Headers.pretty:Pin_Header_Straight_1x04" H 2600 6750 60  0001 C CNN
+F 2 "Socket_Strips.pretty:Socket_Strip_Straight_1x04" H 2600 6750 60  0001 C CNN
 F 3 "" H 2600 6750 60  0000 C CNN
 	1    2600 6750
@@
 F 0 "P14" H 2600 7700 50  0000 C CNN
 F 1 "I2C3" V 2700 7450 50  0000 C CNN
-F 2 "Pin_Headers.pretty:Pin_Header_Straight_1x04" H 2600 7450 60  0001 C CNN
+F 2 "Socket_Strips.pretty:Socket_Strip_Straight_1x04" H 2600 7450 60  0001 C CNN
 F 3 "" H 2600 7450 60  0000 C CNN
 	1    2600 7450
@@
 F 0 "P18" H 5150 5950 50  0000 C CNN
 F 1 "TYP1_GPIO1" V 5250 5600 50  0000 C CNN
-F 2 "Pin_Headers.pretty:Pin_Header_Straight_1x06" H 5150 5600 60  0001 C CNN
+F 2 "Socket_Strips.pretty:Socket_Strip_Straight_1x06" H 5150 5600 60  0001 C CNN
 F 3 "" H 5150 5600 60  0000 C CNN
 	1    5150 5600
@@
 F 0 "P19" H 5150 6850 50  0000 C CNN
 F 1 "TYP1_GPIO2" V 5250 6500 50  0000 C CNN
-F 2 "Pin_Headers.pretty:Pin_Header_Straight_1x06" H 5150 6500 60  0001 C CNN
+F 2 "Socket_Strips.pretty:Socket_Strip_Straight_1x06" H 5150 6500 60  0001 C CNN
 F 3 "" H 5150 6500 60  0000 C CNN
 	1    5150 6500
@@
 F 0 "P20" H 5150 7750 50  0000 C CNN
 F 1 "TYP1_GPIO3" V 5250 7400 50  0000 C CNN
-F 2 "Pin_Headers.pretty:Pin_Header_Straight_1x06" H 5150 7400 60  0001 C CNN
+F 2 "Socket_Strips.pretty:Socket_Strip_Straight_1x06" H 5150 7400 60  0001 C CNN
 F 3 "" H 5150 7400 60  0000 C CNN
 	1    5150 7400
@@
 F 0 "P17" H 4250 3950 50  0000 C CNN
 F 1 "TYP3_UART6" V 4350 3600 50  0000 C CNN
-F 2 "Pin_Headers.pretty:Pin_Header_Straight_1x06" H 4250 3600 60  0001 C CNN
+F 2 "Socket_Strips.pretty:Socket_Strip_Straight_1x06" H 4250 3600 60  0001 C CNN
 F 3 "" H 4250 3600 60  0000 C CNN
 	1    4250 3600
@@
 F 0 "P16" H 4250 3050 50  0000 C CNN
 F 1 "TYP3_UART2" V 4350 2700 50  0000 C CNN
-F 2 "Pin_Headers.pretty:Pin_Header_Straight_1x06" H 4250 2700 60  0001 C CNN
+F 2 "Socket_Strips.pretty:Socket_Strip_Straight_1x06" H 4250 2700 60  0001 C CNN
 F 3 "" H 4250 2700 60  0000 C CNN
 	1    4250 2700
@@
 F 0 "P15" H 4250 2150 50  0000 C CNN
 F 1 "TYP3_UART1" V 4350 1800 50  0000 C CNN
-F 2 "Pin_Headers.pretty:Pin_Header_Straight_1x06" H 4250 1800 60  0001 C CNN
+F 2 "Socket_Strips.pretty:Socket_Strip_Straight_1x06" H 4250 1800 60  0001 C CNN
 F 3 "" H 4250 1800 60  0000 C CNN
 	1    4250 1800
@@
 F 0 "P21" H 6150 2100 50  0000 C CNN
 F 1 "TIM1" H 6150 1400 50  0000 C CNN
-F 2 "Pin_Headers.pretty:Pin_Header_Straight_2x06" H 6150 550 60  0001 C CNN
+F 2 "Socket_Strips.pretty:Socket_Strip_Straight_2x06" H 6150 550 60  0001 C CNN
 F 3 "" H 6150 550 60  0000 C CNN
 	1    6150 1750
@@
 F 0 "P11" H 2600 4900 50  0000 C CNN
 F 1 "TYP2_SPI4" V 2700 4550 50  0000 C CNN
-F 2 "Pin_Headers.pretty:Pin_Header_Straight_1x06" H 2600 4550 60  0001 C CNN
+F 2 "Socket_Strips.pretty:Socket_Strip_Straight_1x06" H 2600 4550 60  0001 C CNN
 F 3 "" H 2600 4550 60  0000 C CNN
 	1    2600 4550
@@
 F 0 "P22" H 6400 5950 50  0000 C CNN
 F 1 "TYP1_GPIO4" V 6500 5600 50  0000 C CNN
-F 2 "Pin_Headers.pretty:Pin_Header_Straight_1x06" H 6400 5600 60  0001 C CNN
+F 2 "Socket_Strips.pretty:Socket_Strip_Straight_1x06" H 6400 5600 60  0001 C CNN
 F 3 "" H 6400 5600 60  0000 C CNN
 	1    6400 5600
@@
 F 0 "P23" H 6400 6850 50  0000 C CNN
 F 1 "TYP1_GPIO5" V 6500 6500 50  0000 C CNN
-F 2 "Pin_Headers.pretty:Pin_Header_Straight_1x06" H 6400 6500 60  0001 C CNN
+F 2 "Socket_Strips.pretty:Socket_Strip_Straight_1x06" H 6400 6500 60  0001 C CNN
 F 3 "" H 6400 6500 60  0000 C CNN
 	1    6400 6500
